Commit message: Object sets: sharedObject becomes reward-only, add non-scored props
The cup/brush task has BOTH hands manipulating the brush, with the cup as a
passive receptacle it is placed into. That is what _object_reward_shares was
written for (one body, two hands, credited once), but sharedObject also deleted
the second body from the scene, leaving the brush nothing to be placed into.

Split the flag's two jobs:
  - collapsing the two scored actors into one is now INFERRED from both sides
    resolving to the same body (two overlapping copies is never a valid scene)
  - sharedObject keeps only the reward split
  - a non-scored prop is declared by the object set, spawned as a free rigid
    body and placed on reset (not teleported per-step, which would push force
    through its contact with the manipulated body)

New main/dataset/object_sets.py is the single registry for both paths: offline
the loaders infer the set from what the capture recorded, live objectSet names
it (there is no pkl to infer from). It also absorbs the block both loaders
duplicated behind "KEEP IDENTICAL" comments, and object names are matched by
name rather than by position in obj_ids, which silently swapped the hands if
Motive reordered.

Fixes a 5 cm scene lift for cup_brush: RECENTER_FINE places the anchor's ORIGIN
above the table, and 0.05 was tuned for bottle_body, whose origin sits 4.88 cm
above its own base. The cup's origin IS its base, so the same lift floated the
hands and both objects. recenter_fine is now per-set; bottle is unchanged.

Verified: loader output is bitwise identical across 14 entries / 6 existing
captures, so the 223 bottle captures and the LOO runs are untouched. Live
bottle regression unchanged (two scored actors, no prop); live and offline
cup_brush both boot with one scored actor plus the cup prop.

Assets: cup/square_brush COACD meshes + urdfs regenerated after the Cup -> cup
rename; resolve_obj_assets now accepts .obj or .ply for the visual mesh.

File: data/my_dataset/obj_files/coacd/cup.urdf (robot description, URDF)
Before this commit: robot square_brush, 1 links, 0 joints
Links:
- link base: geometry collision mesh filename=cup.obj scale=1 1 1; visual mesh filename=cup.obj scale=1 1 1
